File: PCB/FPGC4IOboardV2/FPGC4IOboard.kicad_pcb (KiCad board)
At the start: 4 copper layers, 105.4 x 137.7 mm, 170 parts, among them J1 Conn_PS2_Mini_Din_6, J10 Conn_GPIO_Ext, J11 Conn_SPI_Ext, J12 Conn_Headphone_Jack, J13 Conn_W5500_1, J14 Conn_W5500_2, J15 USB_B_Mini, J16 USB_B_Mini, J2 Conn_SNES, J3 Conn_RGBs, J4 Conn_NConfig, J5 Conn_VGA, J6 Conn_Stacked_USB, J7 Conn_Debug_U8, J8 Conn_Debug_U7, J9 Conn_UART_Ext, Q1 BSS138, Q2 BSS138, Q3 BC847, Q4 BC847, SW1 SW_Push_Rst, SW2 SW_Slide, SW3 SW_Push_Config, SW4 SW_Power, U1 ADV7123, U10 FT232RL, U11 FT232RL, U2 CH376T, U3 CH376T, U4 Conn_02x32_U7, U5 Conn_02x32_U8, U6 ADV7123, U7 W25Q128JVS, U8 ESP32-WROOM-32U, U9 UDA1334ATS, Y1 12MHz, Y2 12MHz

Commit message: Finished V2.0 of the PCB. Send order to JLCPCB.
Routing:
- net Net-(J4-Pad1): track 6.74 -> 141.4 mm, vias 0 -> 5
- net Net-(D2-Pad1): track 0.00 -> 132.3 mm, vias 0 -> 2
- net Net-(D1-Pad1): track 0.00 -> 126.6 mm, vias 0 -> 2
- net Net-(D4-Pad1): track 9.77 -> 132.7 mm, vias 1 -> 3
- net Net-(D3-Pad1): track 8.75 -> 126.6 mm, vias 1 -> 3
- net Net-(C43-Pad2): track 3.48 -> 120.9 mm, vias 0 -> 2
- net Net-(C49-Pad2): track 3.33 -> 113.0 mm, vias 0 -> 3
- net +5V: track 276.5 -> 314.6 mm, vias 2 -> 4
- net GND: track 256.2 -> 258.6 mm, vias 84 -> 85
Other:
- board text added: "Audio Out"
- board text added: "B4RT"
- board text added: "Design by"
- board text added: "Power/Data"
- board text added: "SPI Flash"
- board text removed: "K21"
- board text removed: "TODO: some text or art here"
